File: KiCad/pulsoximeter.kicad_pcb (KiCad board)
At the start: 2 copper layers, 100 x 100 mm, 23 parts, among them J5 Analog, J7 Digital, Q1 DMG2305UX-13, Q2 2N3906C, Q3 2N3906C, SW1 SW_Push, SW2 Display_Button, SW3 Display_Button_2, U2 PicoW

Commit message: Added cool logos to the PCB and generated Gerbers
Parts:
- added G***: LOGO, RPi_Pico:pulsoximeter_logo, B.Cu at (62.9, 136.5)
- added G***: LOGO, RPi_Pico:VDE_Logo, B.Cu at (90.2, 59.1)
- added G***: LOGO, RPi_Pico:ETV_Logo, B.Cu at (57.8, 59.1)
- moved BT1 0.63 mm to (73.7, 99.7)
Other:
- board text added: "+"
- board text added: "3V3"
- board text added: "GND"
- board text added: "Pulsoximeter Example Board V1 www.etv-darmstadt.org/de"
- board text added: "SCL"
- board text added: "SDA"
- board text added: "VSYS"
